File: KiCad OPEN ECU/Connectors.kicad_sch (KiCad schematic)
At the start: 2 parts, among them J1 Delphi_Sicma_24, J2 Delphi_Sicma_24

Commit message: Add files via upload
Parts:
- added U15: ~, AeonLabs_Connectors:121 pin ECU connector header, symbol AeonLabs_connectors:ECU_121_pin_pcb_header_connector
Changed lines of the file:
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@@
     (stroke (width 0) (type default))
   )
-  (wire (pts (xy 138.43 68.58) (xy 142.24 68.58))
+  (wire (pts (xy 146.812 47.879) (xy 150.622 47.879))
     (stroke (width 0) (type default))
   )
@@
     (stroke (width 0) (type default))
   )
-  (wire (pts (xy 142.24 60.96) (xy 138.43 60.96))
+  (wire (pts (xy 150.622 40.259) (xy 146.812 40.259))
     (stroke (width 0) (type default))
   )
@@
     (stroke (width 0) (type default))
   )
-  (wire (pts (xy 142.24 66.04) (xy 138.43 66.04))
-    (stroke (width 0) (type default))
-  )
-  (wire (pts (xy 138.43 63.5) (xy 142.24 63.5))
+  (wire (pts (xy 150.622 45.339) (xy 146.812 45.339))
+    (stroke (width 0) (type default))
+  )
+  (wire (pts (xy 146.812 42.799) (xy 150.622 42.799))
     (stroke (width 0) (type default))
   )
@@
     )
   )
-  (global_label "STEPPER-A1" (shape input) (at 142.24 63.5 0) (fields_autoplaced)
-    (effects (font (size 1.27 1.27)) (justify left))
-    (property "Intersheetrefs" "${INTERSHEET_REFS}" (at 156.6472 63.5 0)
+  (global_label "STEPPER-A1" (shape input) (at 150.622 42.799 0) (fields_autoplaced)
+    (effects (font (size 1.27 1.27)) (justify left))
+    (property "Intersheetrefs" "${INTERSHEET_REFS}" (at 165.0292 42.799 0)
       (effects (font (size 1.27 1.27)) (justify left) hide)
     )
@@
     )
   )
-  (global_label "STEPPER-A2" (shape input) (at 142.24 60.96 0) (fields_autoplaced)
-    (effects (font (size 1.27 1.27)) (justify left))
-    (property "Intersheetrefs" "${INTERSHEET_REFS}" (at 156.6472 60.96 0)
+  (global_label "STEPPER-A2" (shape input) (at 150.622 40.259 0) (fields_autoplaced)
+    (effects (font (size 1.27 1.27)) (justify left))
+    (property "Intersheetrefs" "${INTERSHEET_REFS}" (at 165.0292 40.259 0)
       (effects (font (size 1.27 1.27)) (justify left) hide)
     )
@@
     )
   )
-  (global_label "STEPPER-B2" (shape input) (at 142.24 68.58 0) (fields_autoplaced)
-    (effects (font (size 1.27 1.27)) (justify left))
-    (property "Intersheetrefs" "${INTERSHEET_REFS}" (at 156.8286 68.58 0)
-      (effects (font (size 1.27 1.27)) (justify left) hide)
-    )
-  )
-  (global_label "IDLE-OUT" (shape input) (at 138.43 66.04 180) (fields_autoplaced)
-    (effects (font (size 1.27 1.27)) (justify right))
-    (property "Intersheetrefs" "${INTERSHEET_REFS}" (at 126.9255 66.04 0)
+  (global_label "STEPPER-B2" (shape input) (at 150.622 47.879 0) (fields_autoplaced)
+    (effects (font (size 1.27 1.27)) (justify left))
+    (property "Intersheetrefs" "${INTERSHEET_REFS}" (at 165.2106 47.879 0)
+      (effects (font (size 1.27 1.27)) (justify left) hide)
+    )
+  )
+  (global_label "IDLE-OUT" (shape input) (at 146.812 45.339 180) (fields_autoplaced)
+    (effects (font (size 1.27 1.27)) (justify right))
+    (property "Intersheetrefs" "${INTERSHEET_REFS}" (at 135.3075 45.339 0)
       (effects (font (size 1.27 1.27)) (justify right) hide)
     )
@@
     )
   )
-  (global_label "STEPPER-B1" (shape input) (at 142.24 66.04 0) (fields_autoplaced)
-    (effects (font (size 1.27 1.27)) (justify left))
-    (property "Intersheetrefs" "${INTERSHEET_REFS}" (at 156.8286 66.04 0)
+  (global_label "STEPPER-B1" (shape input) (at 150.622 45.339 0) (fields_autoplaced)
+    (effects (font (size 1.27 1.27)) (justify left))
+    (property "Intersheetrefs" "${INTERSHEET_REFS}" (at 165.2106 45.339 0)
       (effects (font (size 1.27 1.27)) (justify left) hide)
     )
@@
     )
   )
-  (global_label "SPARE1-OUT" (shape input) (at 138.43 60.96 180) (fields_autoplaced)
-    (effects (font (size 1.27 1.27)) (justify right))
-    (property "Intersheetrefs" "${INTERSHEET_REFS}" (at 123.7808 60.96 0)
+  (global_label "SPARE1-OUT" (shape input) (at 146.812 40.259 180) (fields_autoplaced)
+    (effects (font (size 1.27 1.27)) (justify right))
+    (property "Intersheetrefs" "${INTERSHEET_REFS}" (at 132.1628 40.259 0)
       (effects (font (size 1.27 1.27)) (justify right) hide)
     )
@@
     )
   )
-  (global_label "SPARE2-OUT" (shape input) (at 138.43 68.58 180) (fields_autoplaced)
-    (effects (font (size 1.27 1.27)) (justify right))
-    (property "Intersheetrefs" "${INTERSHEET_REFS}" (at 123.7808 68.58 0)
+  (global_label "SPARE2-OUT" (shape input) (at 146.812 47.879 180) (fields_autoplaced)
+    (effects (font (size 1.27 1.27)) (justify right))
+    (property "Intersheetrefs" "${INTERSHEET_REFS}" (at 132.1628 47.879 0)
       (effects (font (size 1.27 1.27)) (justify right) hide)
     )
@@
     )
   )
-  (global_label "VVT-OUT" (shape input) (at 138.43 63.5 180) (fields_autoplaced)
-    (effects (font (size 1.27 1.27)) (justify right))
-    (property "Intersheetrefs" "${INTERSHEET_REFS}" (at 127.8326 63.5 0)
+  (global_label "VVT-OUT" (shape input) (at 146.812 42.799 180) (fields_autoplaced)
+    (effects (font (size 1.27 1.27)) (justify right))
+    (property "Intersheetrefs" "${INTERSHEET_REFS}" (at 136.2146 42.799 0)
       (effects (font (size 1.27 1.27)) (justify right) hide)
     )
@@
         )
       )
+    )
+  )
+  (symbol (lib_id "AeonLabs_connectors:ECU_121_pin_pcb_header_connector") (at 142.494 133.5024 0) (unit 1)
+    (in_bom yes) (on_board yes) (dnp no)
+    (property "Reference" "U15" (at 151.7904 104.4448 0)
+      (effects (font (size 1.27 1.27)))
+    )
+    (property "Value" "~" (at 68.834 104.1908 0)
+      (effects (font (size 1.27 1.27)))
+    )
+    (property "Footprint" "AeonLabs_Connectors:121 pin ECU connector header" (at 144.9324 104.6226 0)
+      (effects (font (size 1.27 1.27)) hide)
+    )
+    (property "Datasheet" "" (at 68.834 104.1908 0)
+      (effects (font (size 1.27 1.27)) hide)
+    )
+    (pin "1")
+    (pin "10")
+    (pin "100")
+    (pin "101")
+    (pin "102")
+    (pin "103")
+    (pin "104")
+    (pin "105")
+    (pin "106")
+    (pin "107")
+    (pin "108")
+    (pin "109")
+    (pin "11")
+    (pin "110")
+    (pin "111")
+    (pin "112")
+    (pin "113")
+    (pin "114")
+    (pin "115")
+    (pin "116")
+    (pin "117")
+    (pin "118")
+    (pin "119")
+    (pin "12")
+    (pin "120")
+    (pin "121")
+    (pin "13")
+    (pin "14")
+    (pin "15")
+    (pin "16")
+    (pin "17")
+    (pin "18")
+    (pin "19")
+    (pin "2")
+    (pin "20")
+    (pin "21")
+    (pin "22")
+    (pin "23")
+    (pin "24")
+    (pin "25")
+    (pin "26")
+    (pin "27")
+    (pin "28")
+    (pin "29")
+    (pin "3")
+    (pin "30")
+    (pin "31")
+    (pin "32")
+    (pin "33")
+    (pin "34")
+    (pin "35")
+    (pin "36")
+    (pin "37")
+    (pin "38")
+    (pin "39")
+    (pin "4")
+    (pin "40")
+    (pin "41")
+    (pin "42")
+    (pin "43")
+    (pin "44")
+    (pin "45")
+    (pin "46")
+    (pin "47")
+    (pin "48")
+    (pin "49")
+    (pin "5")
+    (pin "50")
+    (pin "51")
+    (pin "52")
+    (pin "53")
+    (pin "54")
+    (pin "55")
+    (pin "56")
+    (pin "57")
+    (pin "58")
+    (pin "59")
+    (pin "6")
+    (pin "60")
+    (pin "61")
+    (pin "62")
+    (pin "63")
+    (pin "64")
+    (pin "65")
+    (pin "66")
+    (pin "67")
+    (pin "68")
+    (pin "69")
+    (pin "7")
+    (pin "70")
+    (pin "71")
+    (pin "72")
+    (pin "73")
+    (pin "74")
+    (pin "75")
+    (pin "76")
+    (pin "77")
+    (pin "78")
+    (pin "79")
+    (pin "8")
+    (pin "80")
+    (pin "81")
+    (pin "82")
+    (pin "83")
+    (pin "84")
+    (pin "85")
+    (pin "86")
+    (pin "87")
+    (pin "88")
+    (pin "89")
+    (pin "9")
+    (pin "90")
+    (pin "91")
+    (pin "92")
+    (pin "93")
+    (pin "94")
+    (pin "95")
+    (pin "96")
+    (pin "97")
+    (pin "98")
+    (pin "99")
+    (instances
+      (project "OEM_ECU"
+        (path "/ebe274a6-1c43-4fa2-9d2a-7756c5a7217c/00000000-0000-0000-0000-00005cb197c8"
+          (reference "U15") (unit 1)
+        )
+      )
