File: KiCad OPEN ECU/OEM_ECU.kicad_pcb (KiCad board)
At the start: 2 copper layers, 148.9 x 117.1 mm, 255 parts, among them IC1 MAX9926UAEE_V+, IC2 ZXMS6006DT8, IC3 ZXMS6006DT8, IC4 ZXMS6006DT8, J3 EBC05DRXN, J4 Conn_01x04, J5 TYPE-C-31-M-12, Q1 Q_PNP_BCEC, Q2 Q_DUAL_NMOS_S1G1D2S2G2D1, Q3 Q_DUAL_NMOS_S1G1D2S2G2D1, SW1 219-2MSTR, SW2 219-2MSTR, SW3 219-2MSTR, SW4 219-2MSTR, SW5 SW_DPDT_x2, U1 ESP32C3, U10 SP720, U11 74AHC1G32, U12 TC4424A, U13 LMV324LIDT, U14 W25Q32JVSS, U16 ATSHA204A-MAHDA-T, U18 KP234, U19 MCP2562-E-SN, U2 MC33814, U20 LMV324LIDT, U3 TC4424A, U4 TC4424A, U5 MC33810, U6 MC33810, U7 TC4424A, U8 TC4424A, U9 ADXL343

Commit message: Add files via upload
Parts:
- removed the REF** at (112.3, 38.2)
- added U15: ~, AeonLabs_Connectors:121 pin ECU connector header, F.Cu at (112.3, 38.2)
- moved G*** 2.50 mm to (52.5, 141.3)
Routing:
- net VMM: track 52.1 -> 146.6 mm, vias 2 -> 5
- net GND: track 979.8 -> 1049.4 mm, vias 148 -> 160
- net SPARE2-OUT: track 133.3 -> 184.7 mm, vias 7 -> 8
- net IDLE-OUT: track 134.2 -> 182.3 mm, vias 5 -> 6
- net SPARE1-OUT: track 138.0 -> 183.3 mm
- net STEPPER-A1: track 141.2 -> 182.3 mm
- net IGN4: track 48.7 -> 86.4 mm, vias 1 -> 2
- net FUELPUMP-OUT: track 81.9 -> 106.4 mm
- net IGN7: track 49.6 -> 72.9 mm, vias 1 -> 2
- net IGN8: track 54.9 -> 75.0 mm, vias 1 -> 2
- net IGN3: track 97.6 -> 80.0 mm, vias 3 -> 2
- net IGN5: track 20.9 -> 37.3 mm, vias 0 -> 2
- net IGN1: track 22.1 -> 37.7 mm, vias 0 -> 2
- net FAN-OUT: track 79.1 -> 92.9 mm, vias 5 -> 4
- net IGN6: track 23.8 -> 36.7 mm, vias 1 -> 0
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Other:
- board text added: "Bi-Fuel up to 4 injectors"
- board text added: "up to 8 injectors"

Commit message: Add files via upload
Parts:
- added R70: TC33X-2-503G, AeonLabs_Power:Trimmer potentiometer 3x3mm _TC33X-2-503G, F.Cu at (45.3, 78.4)
- moved J4 8.57 mm to (213.1, 137.4)
- moved G*** 5.00 mm to (49.3, 82.4)
- moved DRVR3 1.18 mm to (51.1, 60.7)
- moved DRVC3 1.18 mm to (49.8, 74.7)
- moved DRVR1 1.18 mm to (49.8, 77.8)
- moved DRVR2 1.18 mm to (49.8, 76.2)
- moved DRVC1 1.18 mm to (45.0, 61.8)
- moved DRVC2 1.18 mm to (48.3, 61.8)
- moved DRV8 1.18 mm to (47.4, 68.3)
- moved G*** 1.12 mm to (138.4, 141.0)
Connections:
- AUC1 pad 2: +3V3 -> 3V3_ESP
- AUR_C1 pad 1: +3V3 -> 3V3_ESP
- AUR_R2 pad 1: +3V3 -> 3V3_ESP
- AUR_l1 pad 1: +3V3 -> 3V3_ESP
- C24 pad 2: +3V3 -> 3V3_ESP
- C31 pad 1: +3V3 -> 3V3_ESP
- D13 pad 2: +3V3 -> 3V3_ESP
- DRV8 pad 15: +3V3 -> 3V3_ESP
- DRV8 pad 16: +3V3 -> 3V3_ESP
- DRV8 pad 17: +3V3 -> 3V3_ESP
- DRVC3 pad 1: +3V3 -> 3V3_ESP
- DRVR2 pad 2: +3V3 -> 3V3_ESP
- EC14 pad 1: 3V3 -> 3V3_ESP
- EC15 pad 1: 3V3 -> 3V3_ESP
- EC16 pad 2: 3V3 -> 3V3_ESP
- EC17 pad 2: 3V3 -> 3V3_ESP
- EC6 pad 1: 3V3 -> 3V3_ESP
- EC7 pad 1: 3V3 -> 3V3_ESP
- EC9 pad 1: 3V3 -> 3V3_ESP
- ER1 pad 1: 3V3 -> 3V3_ESP
- ER3 pad 1: 3V3 -> 3V3_ESP
- ICSP1 pad 1: +3V3 -> 3V3_ESP
- L1 pad 1: 3V3 -> 3V3_ESP
- MCU1 pad E5: +3V3 -> 3V3_ESP
- MCU1 pad E6: +3V3 -> 3V3_ESP
- MCU1 pad E7: +3V3 -> 3V3_ESP
- MCU1 pad E8: +3V3 -> 3V3_ESP
- MCU1 pad F5: +3V3 -> 3V3_ESP
- MCU1 pad F8: +3V3 -> 3V3_ESP
- MCU1 pad G1: +3V3 -> 3V3_ESP
- MKC1 pad 2: +3V3 -> 3V3_ESP
- MKC2 pad 2: +3V3 -> 3V3_ESP
- MKC3 pad 2: +3V3 -> 3V3_ESP
- MKC4 pad 2: +3V3 -> 3V3_ESP
- MKL1 pad 2: +3V3 -> 3V3_ESP
- Q2 pad 2: +3V3 -> 3V3_ESP
- Q2 pad 5: +3V3 -> 3V3_ESP
- Q3 pad 2: +3V3 -> 3V3_ESP
- Q3 pad 5: +3V3 -> 3V3_ESP
- R15 pad 1: +3V3 -> 3V3_ESP
- R17 pad 2: +3V3 -> 3V3_ESP
- R18 pad 2: +3V3 -> 3V3_ESP
- R19 pad 2: +3V3 -> 3V3_ESP
- R48 pad 2: +3V3 -> 3V3_ESP
- R49 pad 1: +3V3 -> 3V3_ESP
- R60 pad 2: +3V3 -> 3V3_ESP
- R61 pad 2: +3V3 -> 3V3_ESP
- REF** pad 1: (no net) -> GND
- TP1 pad 1: +3V3 -> 3V3_ESP
- U1 pad 11: 3V3 -> 3V3_ESP
- U1 pad 17: 3V3 -> 3V3_ESP
- U1 pad 31: 3V3 -> 3V3_ESP
- U1 pad 32: 3V3 -> 3V3_ESP
- U10 pad 16: +3V3 -> 3V3_ESP
- U11 pad 5: +3V3 -> 3V3_ESP
- U14 pad 3: +3V3 -> 3V3_ESP
- U14 pad 7: +3V3 -> 3V3_ESP
- U14 pad 8: +3V3 -> 3V3_ESP
- U16 pad 8: +3V3 -> 3V3_ESP
- U19 pad 5: +3V3 -> 3V3_ESP
- U5 pad 8: +3V3 -> 3V3_ESP
- U6 pad 8: +3V3 -> 3V3_ESP
- U9 pad 1: +3V3 -> 3V3_ESP
- U9 pad 6: +3V3 -> 3V3_ESP
- UART_CON1 pad 1: (no net) -> 3V3_ESP
- UART_CON1 pad 3: (no net) -> TXD0
- UART_CON1 pad 4: (no net) -> RXD0
- UART_CON1 pad 5: (no net) -> ESP_GPIO0_BOOT-DTR
- UART_CON1 pad 6: (no net) -> CHIP_EN
Routing:
- net 3V3_ESP: track 0.00 -> 628.4 mm, vias 0 -> 32
- net +3V3: track 500.9 -> 0.00 mm, vias 23 -> 0
- net SPARE1-OUT: track 183.3 -> 280.1 mm
- net 3V3: track 81.3 -> 0.00 mm, vias 7 -> 0
- net ADC-Clamp-5: track 151.7 -> 226.4 mm
- net ADC-Clamp-6: track 130.8 -> 205.1 mm, vias 3 -> 4
- net 12V-SW: track 352.1 -> 420.5 mm, vias 19 -> 21
- net GND: track 1049.4 -> 1102.8 mm, vias 160 -> 371
- net TPS_Sensor: track 89.1 -> 138.0 mm
- net SPARE1_Sensor: track 61.9 -> 110.0 mm
- net SPARE2_Sensor: track 64.8 -> 110.0 mm
- net IAT_Sensor: track 59.1 -> 96.4 mm
- net O2_Sensor: track 95.7 -> 131.7 mm
- net CLT_Sensor: track 67.0 -> 102.2 mm
- net CRANK-IN-: track 88.7 -> 120.3 mm
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
Commit message: Add files via upload
Parts:
- removed J3: EBC05DRXN, Misc:EBC05DRXN
- removed J4: Conn_01x04, Connector_PinHeader_2.54mm:PinHeader_1x04_P2.54mm_Vertical
- removed U11: 74AHC1G32, Package_TO_SOT_SMD:SOT-353_SC-70-5
- added ESP_FLASH1: W25Q32JVUXIQ, AeonLabs_IC:WSON8 FLASH SPI SON127P800X600X80-9N, F.Cu at (149.3, 79.4)
- added IMU2: LSM6DS3, AeonLabs_Sensors:LSM6DS3 Motion Sensor PQFN50P300X250X86-14N, F.Cu at (104.3, 111.2)
- added LED1: LED_GBRC, AeonLabs_Power:LED_1206_3210_RGB_Metric, F.Cu at (127.1, 120.1)
- added U21: AHT20, AeonLabs_Sensors:AHT20 PSON100P300X300X110-6N, F.Cu at (103.0, 123.9)
- C13, C18, C19, C21, C22, C23, C28, C29, C30: footprint Capacitor_SMD:C_0805_2012Metric -> Capacitor_SMD:C_0603_1608Metric
- R12: footprint Resistor_SMD:R_0603_1608Metric_Pad1.05x0.95mm_HandSolder -> Resistor_SMD:R_0603_1608Metric
- R15, R17, R18, R19, R21, R22, R48, R49: footprint Resistor_SMD:R_0805_2012Metric -> Resistor_SMD:R_0603_1608Metric
- R31, R32, R33, R34, R38, R39, R40, R41, R42, R43, R44, R45, R50, R54: footprint Resistor_SMD:R_0805_2012Metric_Pad1.15x1.40mm_HandSolder -> Resistor_SMD:R_0805_2012Metric
- U14: value W25Q32JVSS -> MPXH6400A; footprint Package_SO:SOIC-8_5.23x5.23mm_P1.27mm -> AeonLabs_Sensors:NXP MAP Sensor
- U9: value ADXL343 -> BMP280; footprint Package_LGA:LGA-14_3x5mm_P0.8mm_LayoutBorder1x6y -> AeonLabs_Sensors:XDCR_BMP280
- moved U14 121.9 mm to (61.1, 63.4), turned to 0 degrees
- moved U9 68.0 mm to (103.1, 127.9), turned to 90 degrees
- moved ICSP1 60.9 mm to (136.8, 140.5), turned to 0 degrees
- moved G*** 23.4 mm to (161.4, 136.4)
- moved U16 20.9 mm to (103.3, 117.4), turned to 90 degrees
- moved AUC1 20.6 mm to (103.3, 120.3)
- moved LR1 14.7 mm to (118.4, 126.0)
- moved ER3 3.04 mm to (109.2, 124.8)
- moved EC15 1.47 mm to (110.8, 126.4)
- moved EC2 1.34 mm to (112.2, 114.8)
- moved EC1 1.30 mm to (109.2, 121.5)
- moved EC8 1.28 mm to (118.5, 116.1)
- moved EC9 1.28 mm to (117.4, 113.2)
- moved ER1 1.28 mm to (109.2, 123.0), turned to 180 degrees
- moved L1 1.26 mm to (119.1, 113.4)
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Connections:
- AUC1 pad 2: 3V3_ESP -> +3V3
- AUR_C1 pad 1: 3V3_ESP -> +3V3
- AUR_R2 pad 1: 3V3_ESP -> +3V3
- AUR_l1 pad 1: 3V3_ESP -> +3V3
- C24 pad 2: 3V3_ESP -> +3V3
- C31 pad 1: 3V3_ESP -> +3V3
- D13 pad 2: 3V3_ESP -> +3V3
- DRV8 pad 15: 3V3_ESP -> +3V3
- DRV8 pad 16: 3V3_ESP -> +3V3
- DRV8 pad 17: 3V3_ESP -> +3V3
- DRVC3 pad 1: 3V3_ESP -> +3V3
- DRVR2 pad 2: 3V3_ESP -> +3V3
- EC14 pad 1: 3V3_ESP -> +3V3
- EC15 pad 1: 3V3_ESP -> +3V3
- EC16 pad 2: 3V3_ESP -> +3V3
- EC17 pad 2: 3V3_ESP -> +3V3
- EC2 pad 1: ADC1_CH4 -> XTAL_32K_P
- EC6 pad 1: 3V3_ESP -> +3V3
- EC7 pad 1: 3V3_ESP -> +3V3
- EC9 pad 1: 3V3_ESP -> +3V3
- ECY1 pad 3: ADC1_CH4 -> XTAL_32K_P
- ER1 pad 1: 3V3_ESP -> +3V3
- ER3 pad 1: 3V3_ESP -> +3V3
- ICSP1 pad 1: 3V3_ESP -> +3V3
- L1 pad 1: 3V3_ESP -> +3V3
- MCU1 pad A1: MCU-D3 -> unconnected-(MCU1A-PTD7-PadA1)
- MCU1 pad A4: MCU-D4 -> unconnected-(MCU1A-PTD4/LLWU_P14-PadA4)
- MCU1 pad E5: 3V3_ESP -> +3V3
- MCU1 pad E6: 3V3_ESP -> +3V3
- MCU1 pad E7: 3V3_ESP -> +3V3
- MCU1 pad E8: 3V3_ESP -> +3V3
- MCU1 pad F5: 3V3_ESP -> +3V3
- MCU1 pad F8: 3V3_ESP -> +3V3
- MCU1 pad G1: 3V3_ESP -> +3V3
- MCU1 pad K5: I2C0_SDA -> ESP32_I2C_SDA
- MCU1 pad M4: I2C0_SCL -> ESP32_I2C_SCL
- MKC1 pad 2: 3V3_ESP -> +3V3
- MKC2 pad 2: 3V3_ESP -> +3V3
- MKC3 pad 2: 3V3_ESP -> +3V3
- MKC4 pad 2: 3V3_ESP -> +3V3
- MKL1 pad 2: 3V3_ESP -> +3V3
- Q2 pad 2: 3V3_ESP -> +3V3
- Q2 pad 5: 3V3_ESP -> +3V3
- Q3 pad 2: 3V3_ESP -> +3V3
- Q3 pad 5: 3V3_ESP -> +3V3
- R15 pad 1: 3V3_ESP -> +3V3
- R17 pad 2: 3V3_ESP -> +3V3
- R18 pad 2: 3V3_ESP -> +3V3
- R19 pad 2: 3V3_ESP -> +3V3
- R48 pad 2: 3V3_ESP -> +3V3
- R49 pad 1: 3V3_ESP -> +3V3
- R60 pad 2: 3V3_ESP -> +3V3
- R61 pad 2: 3V3_ESP -> +3V3
- R70 pad 1: 3V3_ESP -> +3V3
- SW3 pad 2A: Net-(J3-PadA1) -> Net-(U14-VOUT)
- TP1 pad 1: 3V3_ESP -> +3V3
- U1 pad 10: ADC2_CH0_SDA -> ESP32_I2C_SDA
- U1 pad 11: 3V3_ESP -> +3V3
- U1 pad 12: SCL -> ESP32_I2C_SCL
- U1 pad 13: unconnected-(U1-MTDO-Pad13) -> CAN_TXD
- U1 pad 14: GPIO08_MISO -> MCU_UART_RTS_RST
- U1 pad 16: GPIO10_SCK -> MCU_UART0_TX
- U1 pad 17: 3V3_ESP -> +3V3
- U1 pad 19: unconnected-(U1-SPIHD-Pad19) -> LED_B_IO05
- U1 pad 20: unconnected-(U1-SPIWP-Pad20) -> LED_G_IO02
- U1 pad 23: unconnected-(U1-SPID-Pad23) -> LED_R_IO04
- U1 pad 31: 3V3_ESP -> +3V3
- U1 pad 32: 3V3_ESP -> +3V3
- U1 pad 4: ADC1_CH4 -> XTAL_32K_P
- U1 pad 6: ADC1_CH2 -> MCU_UART0_RX
- U1 pad 8: ADC1_CH3 -> MCU_UART0_CTS
- U1 pad 9: ADC1_CH4 -> CAN_RXD
- U10 pad 16: 3V3_ESP -> +3V3
- U14 pad 1: MCU-D6 -> unconnected-(U14-Pad1)
- U14 pad 2: MISO -> VDDA
- U14 pad 3: 3V3_ESP -> GND
- U14 pad 4: GND -> Net-(U14-VOUT)
- U14 pad 5: MOSI -> unconnected-(U14-Pad5)
- U14 pad 6: SCLK -> unconnected-(U14-Pad6)
- U14 pad 7: 3V3_ESP -> unconnected-(U14-Pad7)
- U14 pad 8: 3V3_ESP -> unconnected-(U14-Pad8)
- U16 pad 5: GPIO8_I2C_SDA -> ESP32_I2C_SDA
- U16 pad 6: GPIO9_I2C_SCL -> ESP32_I2C_SCL
- U16 pad 8: 3V3_ESP -> +3V3
- U19 pad 1: MCU-D3 -> CAN_TXD
- U19 pad 4: MCU-D4 -> CAN_RXD
- U19 pad 5: 3V3_ESP -> +3V3
- U5 pad 8: 3V3_ESP -> +3V3
- U6 pad 8: 3V3_ESP -> +3V3
- U9 pad 1: 3V3_ESP -> GND
- U9 pad 2: GND -> +3V3
- U9 pad 3: unconnected-(U9-RES-Pad3) -> ESP32_I2C_SDA
- U9 pad 4: GND -> ESP32_I2C_SCL
- U9 pad 6: 3V3_ESP -> +3V3
- U9 pad 7: MCU-D7 -> GND
- U9 pad 8: unconnected-(U9-INT1-Pad8) -> +3V3
- UART_CON1 pad 1: 3V3_ESP -> +3V3
Routing:
- net +3V3: track 0.00 -> 700.1 mm, vias 0 -> 30
- net 3V3_ESP: track 628.4 -> 0.00 mm, vias 32 -> 0
- net Net-(U14-VOUT): track 0.00 -> 146.2 mm, vias 0 -> 4
- net VDDA: track 204.7 -> 344.8 mm, vias 11 -> 14
- net SCLK: track 231.6 -> 140.1 mm, vias 9 -> 7
- net ESP32_I2C_SDA: track 0.00 -> 89.8 mm, vias 0 -> 4
- net MOSI: track 224.6 -> 139.3 mm, vias 7 -> 6
- net ESP32_I2C_SCL: track 0.00 -> 84.5 mm, vias 0 -> 6
- net MCU_UART_RTS_RST: track 56.2 -> 138.2 mm, vias 3 -> 8
- net MCU_UART0_TX: track 32.3 -> 113.8 mm, vias 2 -> 8
- net SPARE1-OUT: track 280.1 -> 198.8 mm
- net MCU-D4: track 78.6 -> 0.00 mm, vias 2 -> 0
- net CAN_RXD: track 0.00 -> 75.0 mm, vias 0 -> 2
- net MCU-D3: track 73.9 -> 0.00 mm, vias 2 -> 0
- net CAN_TXD: track 0.00 -> 70.4 mm, vias 0 -> 2
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Other:
- board text added: "MAP SENSOR"
