File: KiCad OPEN ECU/OEM_ECU.kicad_pcb (KiCad board)
At the start: 2 copper layers, 148.9 x 117.1 mm, 257 parts, among them IC1 MAX9926UAEE_V+, IC2 ZXMS6006DT8, IC3 ZXMS6006DT8, IC4 ZXMS6006DT8, J5 TYPE-C-31-M-12, Q1 Q_PNP_BCEC, Q2 Q_DUAL_NMOS_S1G1D2S2G2D1, Q3 Q_DUAL_NMOS_S1G1D2S2G2D1, SW1 219-2MSTR, SW2 219-2MSTR, SW3 219-2MSTR, SW4 219-2MSTR, SW5 SW_DPDT_x2, U1 ESP32C3, U10 SP720, U12 TC4424A, U13 LMV324LIDT, U14 MPXH6400A, U16 ATSHA204A-MAHDA-T, U18 KP234, U19 MCP2562-E-SN, U2 MC33814, U20 LMV324LIDT, U21 AHT20, U3 TC4424A, U4 TC4424A, U5 MC33810, U6 MC33810, U7 TC4424A, U8 TC4424A, U9 BMP280

Commit message: Add files via upload
Parts:
- moved IMU2 1.92 mm to (102.5, 111.9), turned to 180 degrees
- moved MKR3 1.01 mm to (86.9, 133.0)
- moved MKR2 1.00 mm to (87.0, 134.6)
Routing:
- net MCU-D7: track 42.5 -> 0.00 mm, vias 4 -> 0
- net GND: track 1068.2 -> 1089.8 mm, vias 364 -> 375
- net +3V3: track 700.1 -> 715.8 mm, vias 30 -> 34
- net MOSI: track 139.3 -> 132.2 mm
- net SCLK: track 140.1 -> 134.5 mm
- net ESP32_I2C_SCL: track 84.5 -> 88.5 mm, vias 6 -> 7
- net CHIP_EN: track 34.2 -> 36.6 mm
- net MCU-A9: track 64.2 -> 62.8 mm
- net MCU-D6: track 61.1 -> 59.7 mm
- net MCU-USB-D+: track 7.82 -> 8.97 mm
- net Net-(DRV8-ISENA): track 16.8 -> 15.8 mm
- net MCU-USB-D-: track 5.98 -> 6.97 mm
- net ESP32_I2C_SDA: track 89.8 -> 90.8 mm
- net MISO: track 111.6 -> 110.8 mm, vias 8 -> 7
- net MCU-D8: track 79.3 -> 78.5 mm
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Other:
- board text added: "UART CAM"
- board text added: "UART EMS"
- board text added: "USB-C EMS"
- board text removed: "12v"
- board text removed: "5v"
- board text removed: "vRef"

Commit message: Add files via upload
Parts:
- removed ICSP1: ICSP1, Connector_JST:JST_SH_SM06B-SRSS-TB_1x06-1MP_P1.00mm_Horizontal
- removed SW5: SW_DPDT_x2, Misc:AYZ0202AGRLC
- removed U18: KP234, Misc:KP234
- added JP5: Jumper_NO_Small, Jumper:SolderJumper-2_P1.3mm_Open_Pad1.0x1.5mm, F.Cu at (84.0, 98.9)
- added JP6: Jumper_NO_Small, Jumper:SolderJumper-2_P1.3mm_Open_Pad1.0x1.5mm, F.Cu at (87.9, 98.9)
- added U11: KP234, AeonLabs_Automotive:kp234 barometric sensor, F.Cu at (166.4, 113.7)
- added UART_CON2: UART_CONN, AeonLabs_Connectors:SOIC_clipProgSmall, B.Cu at (137.5, 143.2)
- U5, U6: footprint IC_Automotive:SOIC32-P0.65-33N -> AeonLabs_Automotive:mc33810 SOIC32-P0.65-33N
- moved G*** 75.4 mm to (180.8, 76.2)
- moved REF** 61.3 mm to (180.3, 87.2)
- moved G*** 52.7 mm to (148.8, 141.1)
- moved G*** 13.7 mm to (57.4, 71.4)
- moved F2 7.43 mm to (98.4, 99.5), turned to 90 degrees
- moved C10 7.38 mm to (74.2, 102.3), turned to -90 degrees
- moved U8 3.57 mm to (93.6, 100.3)
- moved U7 2.10 mm to (78.0, 100.3)
- moved G*** 1.41 mm to (162.8, 136.0)
- moved U16 1.34 mm to (103.3, 118.7)
- moved AUC1 1.29 mm to (103.3, 121.7)
- moved IMU2 1.22 mm to (103.0, 113.0)
- moved U21 0.77 mm to (102.9, 124.7)
- moved G*** 0.15 mm to (107.5, 87.6)
Routing:
- net INJ4: track 47.2 -> 66.8 mm, vias 0 -> 1
- net GND: track 1089.8 -> 1108.2 mm, vias 375 -> 374
- net Net-(U11-Vout): track 4.74 -> 19.0 mm, vias 0 -> 2
- net MCU_UART0_TX: track 113.8 -> 125.5 mm, vias 8 -> 9
- net MCU_UART_RTS_RST: track 138.2 -> 148.1 mm
- net MCU_UART0_RX: track 100.7 -> 108.4 mm, vias 7 -> 8
- net +5V: track 331.0 -> 338.2 mm, vias 15 -> 14
- net MCU_UART0_CTS: track 102.5 -> 109.3 mm
- net +3V3: track 715.8 -> 721.3 mm, vias 34 -> 35
- net IGN7: track 72.9 -> 78.3 mm
- net IGN_V+: track 96.1 -> 91.2 mm
- net VDDA: track 344.8 -> 349.3 mm, vias 14 -> 15
- net Net-(U6-GD2): track 5.12 -> 8.79 mm
- net Net-(F2-Pad1): track 11.1 -> 14.8 mm
- net MCU-D25: track 72.7 -> 75.8 mm
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Other:
- board text added: "12v"
- board text added: "5V Bridge"
- board text added: "5v"
- board text added: "HARDWARE"
- board text added: "IGN Voltage"
- board text removed: "SOURCE"
