File: KiCad OPEN ECU/crank-cam.kicad_sch (KiCad schematic)
At the start: 21 parts, among them IC1 MAX9926UAEE_V+, Q2 Q_DUAL_NMOS_S1G1D2S2G2D1, SW1 219-2MSTR, SW2 219-2MSTR, SW4 219-2MSTR

Commit message: Add files via upload
Parts:
- C28, C29, C30: footprint Capacitor_SMD:C_0805_2012Metric -> Capacitor_SMD:C_0603_1608Metric
- R48, R49: footprint Resistor_SMD:R_0805_2012Metric -> Resistor_SMD:R_0603_1608Metric
Changed lines of the file:
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@@
       (effects (font (size 1.27 1.27)))
     )
-    (property "Footprint" "Resistor_SMD:R_0805_2012Metric" (at 99.568 66.04 90)
+    (property "Footprint" "Resistor_SMD:R_0603_1608Metric" (at 99.568 66.04 90)
       (effects (font (size 1.27 1.27)) hide)
     )
@@
       (effects (font (size 1.27 1.27)))
     )
-    (property "Footprint" "Resistor_SMD:R_0805_2012Metric" (at 96.012 88.9 90)
+    (property "Footprint" "Resistor_SMD:R_0603_1608Metric" (at 96.012 88.9 90)
       (effects (font (size 1.27 1.27)) hide)
     )
@@
       (effects (font (size 1.27 1.27)) (justify left))
     )
-    (property "Footprint" "Capacitor_SMD:C_0805_2012Metric" (at 115.2906 54.61 0)
+    (property "Footprint" "Capacitor_SMD:C_0603_1608Metric" (at 115.2906 54.61 0)
       (effects (font (size 1.27 1.27)) hide)
     )
@@
       (effects (font (size 1.27 1.27)) (justify left))
     )
-    (property "Footprint" "Capacitor_SMD:C_0805_2012Metric" (at 111.4552 87.63 0)
+    (property "Footprint" "Capacitor_SMD:C_0603_1608Metric" (at 111.4552 87.63 0)
       (effects (font (size 1.27 1.27)) hide)
     )
@@
       (effects (font (size 1.27 1.27)) (justify left))
     )
-    (property "Footprint" "Capacitor_SMD:C_0805_2012Metric" (at 118.4402 46.99 0)
-      (effects (font (size 1.27 1.27)) hide)
-    )
+    (property "Footprint" "Capacitor_SMD:C_0603_1608Metric" (at 118.4402 46.99 0)
+      (effects (font (size 1.27 1.27)) hide)
+    )
