File: KiCad OPEN ECU/outputs.kicad_sch (KiCad schematic)
At the start: 33 parts, among them IC2 ZXMS6006DT8, IC3 ZXMS6006DT8, IC4 ZXMS6006DT8

Commit message: Add files via upload
Parts:
- removed DRVRV1: R_Potentiometer, symbol Device:R_Potentiometer
- added R70: TC33X-2-503G, AeonLabs_Power:Trimmer potentiometer 3x3mm _TC33X-2-503G, symbol AeonLabs_Power:Trimmer_Potentiometer_3x3mm_TC33X-2-503G
Connections:
- net +3V3: now also R70.1
- net GND: now also R70.3
- net at DRV8.12 (AVREF), DRV8.13 (BVREF): now also R70.2
Changed lines of the file:
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@@
-    )
-  )
-  (symbol (lib_id "Device:R_Potentiometer") (at 48.387 126.1618 0) (unit 1)
-    (in_bom yes) (on_board yes) (dnp no) (fields_autoplaced)
-    (property "Reference" "DRVRV1" (at 45.5422 124.8918 0)
-      (effects (font (size 1.27 1.27)) (justify right))
-    )
-    (property "Value" "R_Potentiometer" (at 45.5422 127.4318 0)
-      (effects (font (size 1.27 1.27)) (justify right))
-    )
-    (property "Footprint" "" (at 48.387 126.1618 0)
-      (effects (font (size 1.27 1.27)) hide)
-    )
-    (property "Datasheet" "~" (at 48.387 126.1618 0)
-      (effects (font (size 1.27 1.27)) hide)
-    )
-    (pin "1")
-    (pin "2")
-    (pin "3")
-    (instances
-      (project "OEM_ECU"
-        (path "/ebe274a6-1c43-4fa2-9d2a-7756c5a7217c/00000000-0000-0000-0000-00005d6863ce"
-          (reference "DRVRV1") (unit 1)
-        )
-      )
     )
   )
@@
     )
   )
-  (symbol (lib_id "power:+3V3") (at 48.387 122.3518 0) (mirror y) (unit 1)
-    (in_bom yes) (on_board yes) (dnp no)
-    (property "Reference" "#PWR051" (at 48.387 126.1618 0)
-      (effects (font (size 1.27 1.27)) hide)
-    )
-    (property "Value" "+3V3" (at 54.2544 122.3518 0)
-      (effects (font (size 1.27 1.27)) (justify left))
-    )
-    (property "Footprint" "" (at 48.387 122.3518 0)
-      (effects (font (size 1.27 1.27)) hide)
-    )
-    (property "Datasheet" "" (at 48.387 122.3518 0)
+  (symbol (lib_id "power:+3V3") (at 44.577 116.078 0) (mirror y) (unit 1)
+    (in_bom yes) (on_board yes) (dnp no)
+    (property "Reference" "#PWR051" (at 44.577 119.888 0)
+      (effects (font (size 1.27 1.27)) hide)
+    )
+    (property "Value" "+3V3" (at 50.4444 116.078 0)
+      (effects (font (size 1.27 1.27)) (justify left))
+    )
+    (property "Footprint" "" (at 44.577 116.078 0)
+      (effects (font (size 1.27 1.27)) hide)
+    )
+    (property "Datasheet" "" (at 44.577 116.078 0)
       (effects (font (size 1.27 1.27)) hide)
     )
@@
     )
   )
-  (symbol (lib_id "power:GND") (at 48.387 129.9718 0) (mirror y) (unit 1)
-    (in_bom yes) (on_board yes) (dnp no)
-    (property "Reference" "#PWR0154" (at 48.387 136.3218 0)
-      (effects (font (size 1.27 1.27)) hide)
-    )
-    (property "Value" "GND" (at 48.9712 130.4544 0)
-      (effects (font (size 1.27 1.27)) (justify right))
-    )
-    (property "Footprint" "" (at 48.387 129.9718 0)
-      (effects (font (size 1.27 1.27)) hide)
-    )
-    (property "Datasheet" "" (at 48.387 129.9718 0)
+  (symbol (lib_id "power:GND") (at 44.577 136.3218 0) (mirror y) (unit 1)
+    (in_bom yes) (on_board yes) (dnp no)
+    (property "Reference" "#PWR0154" (at 44.577 142.6718 0)
+      (effects (font (size 1.27 1.27)) hide)
+    )
+    (property "Value" "GND" (at 45.1612 136.8044 0)
+      (effects (font (size 1.27 1.27)) (justify right))
+    )
+    (property "Footprint" "" (at 44.577 136.3218 0)
+      (effects (font (size 1.27 1.27)) hide)
+    )
+    (property "Datasheet" "" (at 44.577 136.3218 0)
       (effects (font (size 1.27 1.27)) hide)
     )
@@
         )
       )
+    )
+  )
+  (symbol (lib_id "AeonLabs_Power:Trimmer_Potentiometer_3x3mm_TC33X-2-503G") (at 44.577 126.1618 270) (unit 1)
+    (in_bom yes) (on_board yes) (dnp no) (fields_autoplaced)
+    (property "Reference" "R70" (at 40.0812 124.8918 90)
+      (effects (font (size 1.27 1.27)) (justify right))
+    )
+    (property "Value" "TC33X-2-503G" (at 40.0812 127.4318 90)
+      (effects (font (size 1.27 1.27)) (justify right))
+    )
+    (property "Footprint" "AeonLabs_Power:Trimmer potentiometer 3x3mm _TC33X-2-503G" (at 77.5462 127.4826 0)
+      (effects (font (size 1.27 1.27)) (justify bottom) hide)
+    )
+    (property "Datasheet" "" (at 44.577 126.1618 0)
+      (effects (font (size 1.27 1.27)) hide)
+    )
+    (property "MF" "Bourns" (at 49.3268 165.1762 0)
+      (effects (font (size 1.27 1.27)) (justify bottom) hide)
+    )
+    (property "DESCRIPTION" "Res Trimmer 100K Ohm 25% 1/10W 1_Elec_/1_Mech_Turn _3 X 3.8mm_ Foot Print SMD Embossed T/R" (at 71.3232 126.8222 0)
+      (effects (font (size 1.27 1.27)) (justify bottom) hide)
+    )
+    (property "PACKAGE" "Bourns" (at 52.6796 166.7002 0)
+      (effects (font (size 1.27 1.27)) (justify bottom) hide)
+    )
+    (property "PRICE" "None" (at 48.0568 155.3718 0)
+      (effects (font (size 1.27 1.27)) (justify bottom) hide)
+    )
+    (property "Package" "1608 Bourns" (at 54.1782 153.3906 0)
+      (effects (font (size 1.27 1.27)) (justify bottom) hide)
+    )
+    (property "Check_prices" "https://www.snapeda.com/parts/TC33X-2-503G/Bourns/view-part/?ref=eda" (at 59.4868 127.381 0)
+      (effects (font (size 1.27 1.27)) (justify bottom) hide)
+    )
+    (property "Price" "None" (at 46.228 156.8958 0)
+      (effects (font (size 1.27 1.27)) (justify bottom) hide)
+    )
+    (property "SnapEDA_Link" "https://www.snapeda.com/parts/TC33X-2-503G/Bourns/view-part/?ref=snap" (at 62.4586 129.6924 0)
+      (effects (font (size 1.27 1.27)) (justify bottom) hide)
+    )
+    (property "MP" "TC33X-2-503G" (at 56.261 154.0002 0)
+      (effects (font (size 1.27 1.27)) (justify bottom) hide)
+    )
+    (property "Purchase-URL" "https://www.snapeda.com/api/url_track_click_mouser/?unipart_id=1479476&manufacturer=Bourns&part_name=TC33X-2-503G&search_term=None" (at 67.2592 126.5174 0)
+      (effects (font (size 1.27 1.27)) (justify bottom) hide)
+    )
+    (property "Availability" "In Stock" (at 50.3174 154.1018 0)
+      (effects (font (size 1.27 1.27)) (justify bottom) hide)
+    )
+    (property "AVAILABILITY" "Unavailable" (at 52.2986 153.5684 0)
+      (effects (font (size 1.27 1.27)) (justify bottom) hide)
+    )
+    (property "Description" "\n50 kOhms 0.1W, 1/10W J Lead Surface Mount Trimmer Potentiometer Cermet 1.0 Turn Top Adjustment\n" (at 74.8538 124.8918 0)
+      (effects (font (size 1.27 1.27)) (justify bottom) hide)
+    )
+    (pin "2")
+    (pin "3")
+    (pin "1")
+    (instances
+      (project "OEM_ECU"
+        (path "/ebe274a6-1c43-4fa2-9d2a-7756c5a7217c/00000000-0000-0000-0000-00005d6863ce"
+          (reference "R70") (unit 1)
+        )
+      )

Commit message: Add files via upload
Parts:
- R31, R32, R33, R34, R38, R39, R40, R41, R42, R43, R44, R45: footprint Resistor_SMD:R_0805_2012Metric_Pad1.15x1.40mm_HandSolder -> Resistor_SMD:R_0805_2012Metric
Changed lines of the file:
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@@
       (effects (font (size 1.27 1.27)))
     )
-    (property "Footprint" "Resistor_SMD:R_0805_2012Metric_Pad1.15x1.40mm_HandSolder" (at 189.23 112.522 90)
+    (property "Footprint" "Resistor_SMD:R_0805_2012Metric" (at 189.23 112.522 90)
       (effects (font (size 1.27 1.27)) hide)
     )
@@
       (effects (font (size 1.27 1.27)))
     )
-    (property "Footprint" "Resistor_SMD:R_0805_2012Metric_Pad1.15x1.40mm_HandSolder" (at 189.23 117.602 90)
+    (property "Footprint" "Resistor_SMD:R_0805_2012Metric" (at 189.23 117.602 90)
       (effects (font (size 1.27 1.27)) hide)
     )
@@
       (effects (font (size 1.27 1.27)) (justify right))
     )
-    (property "Footprint" "Resistor_SMD:R_0805_2012Metric_Pad1.15x1.40mm_HandSolder" (at 197.358 127 90)
+    (property "Footprint" "Resistor_SMD:R_0805_2012Metric" (at 197.358 127 90)
       (effects (font (size 1.27 1.27)) hide)
     )
@@
       (effects (font (size 1.27 1.27)) (justify right))
     )
-    (property "Footprint" "Resistor_SMD:R_0805_2012Metric_Pad1.15x1.40mm_HandSolder" (at 197.358 106.68 90)
+    (property "Footprint" "Resistor_SMD:R_0805_2012Metric" (at 197.358 106.68 90)
       (effects (font (size 1.27 1.27)) hide)
     )
@@
       (effects (font (size 1.27 1.27)))
     )
-    (property "Footprint" "Resistor_SMD:R_0805_2012Metric_Pad1.15x1.40mm_HandSolder" (at 34.5694 38.1762 90)
+    (property "Footprint" "Resistor_SMD:R_0805_2012Metric" (at 34.5694 38.1762 90)
       (effects (font (size 1.27 1.27)) hide)
     )
@@
       (effects (font (size 1.27 1.27)))
     )
-    (property "Footprint" "Resistor_SMD:R_0805_2012Metric_Pad1.15x1.40mm_HandSolder" (at 34.5694 43.2562 90)
+    (property "Footprint" "Resistor_SMD:R_0805_2012Metric" (at 34.5694 43.2562 90)
       (effects (font (size 1.27 1.27)) hide)
     )
@@
       (effects (font (size 1.27 1.27)) (justify right))
     )
-    (property "Footprint" "Resistor_SMD:R_0805_2012Metric_Pad1.15x1.40mm_HandSolder" (at 42.6974 52.6542 90)
+    (property "Footprint" "Resistor_SMD:R_0805_2012Metric" (at 42.6974 52.6542 90)
       (effects (font (size 1.27 1.27)) hide)
     )
@@
       (effects (font (size 1.27 1.27)) (justify right))
     )
-    (property "Footprint" "Resistor_SMD:R_0805_2012Metric_Pad1.15x1.40mm_HandSolder" (at 42.6974 32.3342 90)
+    (property "Footprint" "Resistor_SMD:R_0805_2012Metric" (at 42.6974 32.3342 90)
       (effects (font (size 1.27 1.27)) hide)
     )
@@
       (effects (font (size 1.27 1.27)))
     )
-    (property "Footprint" "Resistor_SMD:R_0805_2012Metric_Pad1.15x1.40mm_HandSolder" (at 209.7786 40.767 90)
+    (property "Footprint" "Resistor_SMD:R_0805_2012Metric" (at 209.7786 40.767 90)
       (effects (font (size 1.27 1.27)) hide)
     )
@@
       (effects (font (size 1.27 1.27)))
     )
-    (property "Footprint" "Resistor_SMD:R_0805_2012Metric_Pad1.15x1.40mm_HandSolder" (at 209.7786 45.847 90)
+    (property "Footprint" "Resistor_SMD:R_0805_2012Metric" (at 209.7786 45.847 90)
       (effects (font (size 1.27 1.27)) hide)
     )
@@
       (effects (font (size 1.27 1.27)) (justify right))
     )
-    (property "Footprint" "Resistor_SMD:R_0805_2012Metric_Pad1.15x1.40mm_HandSolder" (at 217.9066 55.245 90)
+    (property "Footprint" "Resistor_SMD:R_0805_2012Metric" (at 217.9066 55.245 90)
       (effects (font (size 1.27 1.27)) hide)
     )
@@
       (effects (font (size 1.27 1.27)) (justify right))
     )
-    (property "Footprint" "Resistor_SMD:R_0805_2012Metric_Pad1.15x1.40mm_HandSolder" (at 217.9066 34.925 90)
-      (effects (font (size 1.27 1.27)) hide)
-    )
+    (property "Footprint" "Resistor_SMD:R_0805_2012Metric" (at 217.9066 34.925 90)
+      (effects (font (size 1.27 1.27)) hide)
+    )
