File: KiCad OPEN ECU/comms.kicad_sch (KiCad schematic)
At the start: 10 parts, among them J4 Conn_01x04, U11 74AHC1G32, U14 W25Q32JVSS, U19 MCP2562-E-SN, U9 ADXL343

Commit message: Add files via upload
Parts:
- removed J4: Conn_01x04, Connector_PinHeader_2.54mm:PinHeader_1x04_P2.54mm_Vertical, symbol Connector_Generic:Conn_01x04
- removed U11: 74AHC1G32, Package_TO_SOT_SMD:SOT-353_SC-70-5, symbol 74xGxx:74AHC1G32
- removed U14: W25Q32JVSS, Package_SO:SOIC-8_5.23x5.23mm_P1.27mm, symbol Memory_Flash:W25Q32JVSS
- removed U9: ADXL343, Package_LGA:LGA-14_3x5mm_P0.8mm_LayoutBorder1x6y, symbol Sensor_Motion:ADXL343
- added IMU1: LSM6DS3, AeonLabs_Sensors:LSM6DS3 Motion Sensor PQFN50P300X250X86-14N, symbol Sensor_Motion:LSM6DS3
- added U4: AHT20, AeonLabs_Sensors:AHT20 PSON100P300X300X110-6N, symbol Sensor:AHT20
- added U5: BMP280, AeonLabs_Sensors:XDCR_BMP280, symbol AeonLabs_Sensors:BMP280
- R50, R54: footprint Resistor_SMD:R_0805_2012Metric_Pad1.15x1.40mm_HandSolder -> Resistor_SMD:R_0805_2012Metric
Connections:
- net +3V3: now also IMU1.5 (VDDIO), IMU1.8 (VDD), U4.2 (VDD), U5.2 (CSB), U5.6 (VDDIO), U5.8 (VDD)
- net GND: now also IMU1.6 (GND), IMU1.7 (GND), U4.5 (GND), U5.1 (GND), U5.5 (SDO), U5.7 (GND)
- net MCU-D3 renamed CAN_TXD
- net MCU-D4 renamed CAN_RXD
- new net: U4.1 (NC), U4.6 (NC)
- new net ESP32_I2C_SCL: IMU1.13 (SCL), U4.3 (SCL), U5.4 (SCK)
- new net ESP32_I2C_SDA: IMU1.14 (SDA), U4.4 (SDA), U5.3 (SDI)
- no-connect marks 0 -> 6
Other:
- note added: "Motion Sensor"
- note added: "Temperature and Humidity Sensor"
- note removed: "Accelerometer"
- note removed: "Flash Storage"
- note removed: "HC-05 Bluetooth Connector"
- moved on the sheet: C31, C33, JP1, R50, R54, U19

Commit message: Add files via upload
Other:
- company: (none) -> WWW.AEONLABS.SCIENCE
- title: (none) -> OPEN ECU
Changed lines of the file:
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@@
 (kicad_sch (version 20230121) (generator eeschema)
   (paper "A4")
+  (title_block
+    (title "OPEN ECU")
+    (date "2023-12-14")
+    (rev "12-2023")
+    (company "WWW.AEONLABS.SCIENCE")
+    (comment 1 "https://github.com/aeonSolutions/AeonLabs-AI-Volvo-MKII-Open-Hardware")
+    (comment 2 "Creative Commons Share alike non commercial")
+  )
   (junction (at 80.6958 146.685) (diameter 0) (color 0 0 0 0)
   )
