File: KiCad OPEN ECU/OEM_ECU.kicad_sch (KiCad schematic)
At the start: 46 parts, among them J1 TYPE-C-31-M-12, J6 RFShield_OnePiece, U1 ATSHA204A-MAHDA-T, U1 ESP32C3

Commit message: Add files via upload
Parts:
- UART_CON1: footprint (none) -> AeonLabs_Connectors:SOIC_clipProgSmall
Connections:
- net +3V3: now also EC11.1, EC2.2, EC3.1, EC4.2, EC5.1, EC7.1, EC8.1, ER1.1, ER3.1, L1.1, U1.11 (VDD3P3_RTC), U1.17 (VDD3P3_CPU), U1.31 (VDDA), U1.32 (VDDA__1), UART_CON1.1 (Pin_1)
- net 3V3: no longer EC11.1, EC2.2, EC3.1, EC4.2, EC5.1, EC7.1, EC8.1, ER1.1, ER3.1, L1.1, U1.11 (VDD3P3_RTC), U1.17 (VDD3P3_CPU), U1.31 (VDDA), U1.32 (VDDA__1), UART_CON1.1 (Pin_1)
Changed lines of the file:
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@@
     (stroke (width 0) (type default))
   )
+  (wire (pts (xy 34.925 120.2182) (xy 33.655 120.2182))
+    (stroke (width 0) (type default))
+  )
   (wire (pts (xy 50.1142 82.9056) (xy 42.4942 82.9056))
     (stroke (width 0) (type default))
@@
     )
   )
-  (global_label "3V3" (shape input) (at 33.0962 82.9056 180) (fields_autoplaced)
-    (effects (font (size 1.27 1.27)) (justify right))
-    (property "Intersheetrefs" "${INTERSHEET_REFS}" (at 27.1755 82.8262 0)
-      (effects (font (size 1.27 1.27)) (justify right) hide)
-    )
-  )
   (global_label "MCU-A6" (shape input) (at 275.3106 127.4318 180) (fields_autoplaced)
     (effects (font (size 1.27 1.27)) (justify right))
@@
     )
   )
-  (global_label "3V3" (shape input) (at 193.675 89.2048 0) (fields_autoplaced)
-    (effects (font (size 1.27 1.27)) (justify left))
-    (property "Intersheetrefs" "${INTERSHEET_REFS}" (at 199.5957 89.2842 0)
-      (effects (font (size 1.27 1.27)) (justify left) hide)
-    )
-  )
   (global_label "MCU_UART0_RX" (shape input) (at 199.009 225.4758 0) (fields_autoplaced)
     (effects (font (size 1.27 1.27)) (justify left))
@@
     )
   )
-  (global_label "3V3" (shape input) (at 33.655 120.2182 0) (fields_autoplaced)
-    (effects (font (size 1.27 1.27)) (justify left))
-    (property "Intersheetrefs" "${INTERSHEET_REFS}" (at 39.5757 120.1388 0)
-      (effects (font (size 1.27 1.27)) (justify left) hide)
-    )
-  )
   (global_label "I2C0_SCL" (shape input) (at 355.1682 66.421 0) (fields_autoplaced)
     (effects (font (size 1.27 1.27)) (justify left))
@@
     )
   )
-  (global_label "3V3" (shape input) (at 99.3902 114.554 180) (fields_autoplaced)
-    (effects (font (size 1.27 1.27)) (justify right))
-    (property "Intersheetrefs" "${INTERSHEET_REFS}" (at 93.4695 114.4746 0)
-      (effects (font (size 1.27 1.27)) (justify right) hide)
-    )
-  )
   (global_label "MCU-A8" (shape input) (at 374.1674 203.9112 180) (fields_autoplaced)
     (effects (font (size 1.27 1.27)) (justify right))
@@
     )
   )
+  (symbol (lib_id "power:+3V3") (at 193.675 89.2048 270) (unit 1)
+    (in_bom yes) (on_board yes) (dnp no)
+    (property "Reference" "#PWR0159" (at 189.865 89.2048 0)
+      (effects (font (size 1.27 1.27)) hide)
+    )
+    (property "Value" "+3V3" (at 196.9262 89.5858 90)
+      (effects (font (size 1.27 1.27)) (justify left))
+    )
+    (property "Footprint" "" (at 193.675 89.2048 0)
+      (effects (font (size 1.27 1.27)) hide)
+    )
+    (property "Datasheet" "" (at 193.675 89.2048 0)
+      (effects (font (size 1.27 1.27)) hide)
+    )
+    (pin "1")
+    (instances
+      (project "OEM_ECU"
+        (path "/ebe274a6-1c43-4fa2-9d2a-7756c5a7217c/00000000-0000-0000-0000-00005cfb00f8"
+          (reference "#PWR0159") (unit 1)
+        )
+        (path "/ebe274a6-1c43-4fa2-9d2a-7756c5a7217c"
+          (reference "#PWR078") (unit 1)
+        )
+      )
+    )
+  )
   (symbol (lib_id "Connector:Conn_01x06_Socket") (at 28.575 115.1382 180) (unit 1)
     (in_bom yes) (on_board yes) (dnp no)
@@
       (effects (font (size 1.27 1.27)))
     )
-    (property "Footprint" "" (at 28.575 115.1382 0)
+    (property "Footprint" "AeonLabs_Connectors:SOIC_clipProgSmall" (at 28.575 115.1382 0)
       (effects (font (size 1.27 1.27)) hide)
     )
@@
     )
   )
+  (symbol (lib_id "power:+3V3") (at 34.925 120.2182 270) (unit 1)
+    (in_bom yes) (on_board yes) (dnp no)
+    (property "Reference" "#PWR0159" (at 31.115 120.2182 0)
+      (effects (font (size 1.27 1.27)) hide)
+    )
+    (property "Value" "+3V3" (at 38.1762 120.5992 90)
+      (effects (font (size 1.27 1.27)) (justify left))
+    )
+    (property "Footprint" "" (at 34.925 120.2182 0)
+      (effects (font (size 1.27 1.27)) hide)
+    )
+    (property "Datasheet" "" (at 34.925 120.2182 0)
+      (effects (font (size 1.27 1.27)) hide)
+    )
+    (pin "1")
+    (instances
+      (project "OEM_ECU"
+        (path "/ebe274a6-1c43-4fa2-9d2a-7756c5a7217c/00000000-0000-0000-0000-00005cfb00f8"
+          (reference "#PWR0159") (unit 1)
+        )
+        (path "/ebe274a6-1c43-4fa2-9d2a-7756c5a7217c"
+          (reference "#PWR080") (unit 1)
+        )
+      )
+    )
+  )
   (symbol (lib_id "Interface_USB:TYPE-C-31-M-12") (at 116.5098 152.0952 0) (unit 1)
     (in_bom yes) (on_board yes) (dnp no) (fields_autoplaced)
@@
     )
   )
+  (symbol (lib_id "power:+3V3") (at 33.0962 82.9056 90) (mirror x) (unit 1)
+    (in_bom yes) (on_board yes) (dnp no)
+    (property "Reference" "#PWR0159" (at 36.9062 82.9056 0)
+      (effects (font (size 1.27 1.27)) hide)
+    )
+    (property "Value" "+3V3" (at 29.845 83.2866 90)
+      (effects (font (size 1.27 1.27)) (justify left))
+    )
+    (property "Footprint" "" (at 33.0962 82.9056 0)
+      (effects (font (size 1.27 1.27)) hide)
+    )
+    (property "Datasheet" "" (at 33.0962 82.9056 0)
+      (effects (font (size 1.27 1.27)) hide)
+    )
+    (pin "1")
+    (instances
+      (project "OEM_ECU"
+        (path "/ebe274a6-1c43-4fa2-9d2a-7756c5a7217c/00000000-0000-0000-0000-00005cfb00f8"
+          (reference "#PWR0159") (unit 1)
+        )
+        (path "/ebe274a6-1c43-4fa2-9d2a-7756c5a7217c"
+          (reference "#PWR079") (unit 1)
+        )
+      )
+    )
+  )
   (symbol (lib_id "power:GNDA") (at 202.9206 168.7322 90) (unit 1)
     (in_bom yes) (on_board yes) (dnp no)
@@
         )
       )
+    )
+  )
+  (symbol (lib_id "power:+3V3") (at 99.3902 114.554 90) (mirror x) (unit 1)
+    (in_bom yes) (on_board yes) (dnp no)
+    (property "Reference" "#PWR0159" (at 103.2002 114.554 0)
+      (effects (font (size 1.27 1.27)) hide)
+    )
+    (property "Value" "+3V3" (at 96.139 114.935 90)
+      (effects (font (size 1.27 1.27)) (justify left))
+    )
+    (property "Footprint" "" (at 99.3902 114.554 0)
+      (effects (font (size 1.27 1.27)) hide)
+    )
+    (property "Datasheet" "" (at 99.3902 114.554 0)
+      (effects (font (size 1.27 1.27)) hide)
+    )
+    (pin "1")
+    (instances
+      (project "OEM_ECU"
+        (path "/ebe274a6-1c43-4fa2-9d2a-7756c5a7217c/00000000-0000-0000-0000-00005cfb00f8"
+          (reference "#PWR0159") (unit 1)
+        )
+        (path "/ebe274a6-1c43-4fa2-9d2a-7756c5a7217c"
+          (reference "#PWR077") (unit 1)
+        )
+      )

Commit message: Add files via upload
Parts:
- added ESP_FLASH2: W25Q32JVUXIQ, AeonLabs_IC:WSON8 FLASH SPI SON127P800X600X80-9N, symbol Memory_Flash:SPI_Flash_W25Q128JVS
- LED1: footprint LED_SMD:LED_1206_3210_RGB_Metric -> AeonLabs_Power:LED_1206_3210_RGB_Metric
Connections:
- net 3V3 is gone; now on net +3V3: LED1.4 (K)
- net ADC1_CH2 is gone; now on net MCU_UART0_RX: U1.6 (GPIO2)
- net ADC1_CH3 is gone; now on net MCU_UART0_CTS: U1.8 (GPIO3)
- net GPIO08_MISO is gone; now on net MCU_UART_RTS_RST: U1.14 (GPIO8)
- net GPIO10_SCK is gone; now on net MCU_UART0_TX: U1.16 (GPIO10)
- net GPIO8_I2C_SDA is gone; now on net ESP32_I2C_SDA: U1.5 (SDA)
- net I2C0_SCL is gone; now on net ESP32_I2C_SCL: MCU1.M4 (PTE24)
- net I2C0_SDA is gone; now on net ESP32_I2C_SDA: MCU1.K5 (PTE25)
- net SCL is gone; now on net ESP32_I2C_SCL: U1.12 (MTCK)
- net +3V3: now also ESP_FLASH2.3 (IO2), ESP_FLASH2.7 (IO3), ESP_FLASH2.8 (VCC)
- net GND: now also ESP_FLASH2.4 (GND), ESP_FLASH2.9 (GND)
- net LED_B_IO05: now also U1.19 (SPIHD)
- net LED_G_IO02: now also U1.20 (SPIWP)
- net LED_R_IO04: now also U1.23 (SPID)
- net MCU-D3: no longer MCU1.A1 (PTD7)
- net MCU-D4: no longer MCU1.A4 (PTD4/LLWU_P14)
- net MCU-D6: now also ESP_FLASH2.1 (~{CS})
- net MISO: now also ESP_FLASH2.2 (DO(IO1))
- net MOSI: now also ESP_FLASH2.5 (DI(IO0))
- net SCLK: now also ESP_FLASH2.6 (CLK)
- net CAN_TXD: now reaches U1.13 (MTDO)
- net ADC1_CH4 renamed XTAL_32K_P
- net XTAL_32K_P: no longer U1.9 (MTMS)
- net ADC2_CH0_SDA renamed ESP32_I2C_SDA
- net GPIO9_I2C_SCL renamed ESP32_I2C_SCL
- new net CAN_RXD: U1.9 (MTMS)
- no-connect marks 11 -> 7
Other:
- note added: "16Mbit Flash Memory W25Q32JVUXIQ"
- moved on the sheet: EC2, EC4, ER3, J1, USB_PLUG_R1, USB_PLUG_R3, USB_PLYG_R2

Commit message: Add files via upload
Parts:
- removed ICSP1: ICSP1, Connector_JST:JST_SH_SM06B-SRSS-TB_1x06-1MP_P1.00mm_Horizontal, symbol Connector:Conn_01x06_Socket
- added UART_CON2: UART_CONN, AeonLabs_Connectors:SOIC_clipProgSmall, symbol Connector:Conn_01x06_Socket
Connections:
- net +3V3: now also UART_CON2.1 (Pin_1)
- net GND: now also UART_CON2.2 (Pin_2)
- net MCU_UART0_CTS: now also UART_CON2.5 (Pin_5)
- net MCU_UART0_RX: now also UART_CON2.4 (Pin_4)
- net MCU_UART0_TX: now also UART_CON2.3 (Pin_3)
- net MCU_UART_RTS_RST: now also UART_CON2.6 (Pin_6)
Changed lines of the file:
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@@
+    )
+  )
+  (symbol (lib_id "Connector:Conn_01x06_Socket") (at 193.929 228.0158 180) (unit 1)
+    (in_bom yes) (on_board yes) (dnp no)
+    (property "Reference" "UART_CON2" (at 189.357 229.1588 90)
+      (effects (font (size 1.27 1.27)))
+    )
+    (property "Value" "UART_CONN" (at 191.9986 228.4476 90)
+      (effects (font (size 1.27 1.27)))
+    )
+    (property "Footprint" "AeonLabs_Connectors:SOIC_clipProgSmall" (at 193.929 228.0158 0)
+      (effects (font (size 1.27 1.27)) hide)
+    )
+    (property "Datasheet" "~" (at 193.929 228.0158 0)
+      (effects (font (size 1.27 1.27)) hide)
+    )
+    (pin "1")
+    (pin "2")
+    (pin "3")
+    (pin "4")
+    (pin "5")
+    (pin "6")
+    (instances
+      (project "OEM_ECU"
+        (path "/ebe274a6-1c43-4fa2-9d2a-7756c5a7217c"
+          (reference "UART_CON2") (unit 1)
+        )
+      )
+      (project "ESP32 C3 PCB TEMPLATE"
+        (path "/f1f5a39e-9869-4f00-8f70-65c53b83e907"
+          (reference "UART_CON1") (unit 1)
+        )
+      )
     )
   )
@@
         )
       )
-    )
-  )
-  (symbol (lib_id "Connector:Conn_01x06_Socket") (at 193.929 228.0158 180) (unit 1)
-    (in_bom yes) (on_board yes) (dnp no)
-    (property "Reference" "ICSP1" (at 188.7728 226.7458 0)
-      (effects (font (size 1.27 1.27)))
-    )
-    (property "Value" "ICSP1" (at 189.4586 224.3582 0)
-      (effects (font (size 1.27 1.27)))
-    )
-    (property "Footprint" "Connector_JST:JST_SH_SM06B-SRSS-TB_1x06-1MP_P1.00mm_Horizontal" (at 193.929 228.0158 0)
-      (effects (font (size 1.27 1.27)) hide)
-    )
-    (property "Datasheet" "~" (at 193.929 228.0158 0)
-      (effects (font (size 1.27 1.27)) hide)
-    )
-    (pin "1")
-    (pin "2")
-    (pin "3")
-    (pin "4")
-    (pin "5")
-    (pin "6")
-    (instances
-      (project "LDAD_ATOM _PRO _LCD _ABS_Enclosure_52x48_16bit"
-        (path "/e63e39d7-6ac0-4ffd-8aa3-1841a4541b55"
-          (reference "ICSP1") (unit 1)
-        )
-      )
-      (project "OEM_ECU"
-        (path "/ebe274a6-1c43-4fa2-9d2a-7756c5a7217c"
-          (reference "ICSP1") (unit 1)
-        )
-      )
