File: KiCad OPEN ECU/inputs.kicad_sch (KiCad schematic)
At the start: 41 parts, among them J3 EBC05DRXN, SW1 219-2MSTR, U10 SP720, U13 LMV324LIDT, U18 KP234

Commit message: Add files via upload
Parts:
- removed J3: EBC05DRXN, Misc:EBC05DRXN, symbol Misc:EBC05DRXN
- added U14: MPXH6400A, AeonLabs_Sensors:NXP MAP Sensor, symbol AeonLabs_Sensors:MPXH6400A_MAP_Sensor
- C13, C18, C19, C21, C22, C23: footprint Capacitor_SMD:C_0805_2012Metric -> Capacitor_SMD:C_0603_1608Metric
- R12: footprint Resistor_SMD:R_0603_1608Metric_Pad1.05x0.95mm_HandSolder -> Resistor_SMD:R_0603_1608Metric
- R15, R17, R18, R19, R21, R22: footprint Resistor_SMD:R_0805_2012Metric -> Resistor_SMD:R_0603_1608Metric
Connections:
- net GND: now also U14.3 (GND)
- net VDDA: now also U14.2 (VS)
- net at SW1.2A: now also U14.4 (VOUT)
Other:
- moved on the sheet: SW1

Commit message: Add files via upload
Parts:
- removed U18: KP234, Misc:KP234, symbol Misc:KP234
- added U11: KP234, AeonLabs_Automotive:kp234 barometric sensor, symbol AeonLabs_Automotive:KP234
Connections:
- net GND: now also U11.6 (GND), U11.8 (NC)
- net VDDA: now also U11.5 (Vcc)
- net at R28.1: now also U11.7 (Vout)
Changed lines of the file:
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@@
   (junction (at 93.98 172.72) (diameter 0) (color 0 0 0 0)
   )
-  (junction (at 128.27 54.61) (diameter 0) (color 0 0 0 0)
-  )
   (junction (at 129.54 78.74) (diameter 0) (color 0 0 0 0)
   )
   (junction (at 129.54 38.1) (diameter 0) (color 0 0 0 0)
   )
+  (junction (at 128.27 54.61) (diameter 0) (color 0 0 0 0)
+  )
   (junction (at 64.77 74.93) (diameter 0) (color 0 0 0 0)
   )
@@
     (stroke (width 0) (type default))
   )
-  (wire (pts (xy 127 54.61) (xy 128.27 54.61))
-    (stroke (width 0) (type default))
-  )
   (wire (pts (xy 260.35 72.39) (xy 257.81 72.39))
     (stroke (width 0) (type default))
@@
     (stroke (width 0) (type default))
   )
+  (wire (pts (xy 127 54.61) (xy 128.27 54.61))
+    (stroke (width 0) (type default))
+  )
   (wire (pts (xy 128.27 54.61) (xy 133.35 54.61))
     (stroke (width 0) (type default))
@@
     )
   )
-  (symbol (lib_id "Misc:KP234") (at 133.35 46.99 0) (unit 1)
-    (in_bom yes) (on_board yes) (dnp no)
-    (property "Reference" "U18" (at 122.4534 44.6786 0)
+  (symbol (lib_id "AeonLabs_Automotive:KP234") (at 133.35 46.99 0) (unit 1)
+    (in_bom yes) (on_board yes) (dnp no) (fields_autoplaced)
+    (property "Reference" "U11" (at 121.3612 44.45 0)
       (effects (font (size 1.27 1.27)) (justify right))
     )
-    (property "Value" "KP234" (at 122.4534 46.99 0)
+    (property "Value" "KP234" (at 121.3612 46.99 0)
       (effects (font (size 1.27 1.27)) (justify right))
     )
-    (property "Footprint" "Misc:KP234" (at 122.4534 49.3014 0)
+    (property "Footprint" "AeonLabs_Automotive:kp234 barometric sensor" (at 121.3612 49.53 0)
       (effects (font (size 1.27 1.27)) (justify right))
     )
@@
       (effects (font (size 1.27 1.27)) hide)
     )
-    (property "Digikey Part Number" "448-KP234XTMA1CT-ND" (at 133.35 46.99 0)
+    (property "Digikey Part Number" "448-KP234XTMA1CT-ND" (at 152.5524 36.1442 0)
       (effects (font (size 1.27 1.27)) hide)
     )
-    (property "Manufacturer_Name" "Infineon" (at 133.35 46.99 0)
+    (property "Manufacturer_Name" "Infineon" (at 144.5006 34.036 0)
       (effects (font (size 1.27 1.27)) hide)
     )
-    (property "Manufacturer_Part_Number" "KP234XTMA1" (at 133.35 46.99 0)
+    (property "Manufacturer_Part_Number" "KP234XTMA1" (at 156.083 33.6804 0)
       (effects (font (size 1.27 1.27)) hide)
     )
-    (property "URL" "https://www.digikey.com.au/product-detail/en/infineon-technologies/KP234XTMA1/448-KP234XTMA1CT-ND/12718428" (at 133.35 46.99 0)
+    (property "URL" "https://www.digikey.com.au/product-detail/en/infineon-technologies/KP234XTMA1/448-KP234XTMA1CT-ND/12718428" (at 133.1722 26.5684 0)
       (effects (font (size 1.27 1.27)) hide)
     )
@@
       (project "OEM_ECU"
         (path "/ebe274a6-1c43-4fa2-9d2a-7756c5a7217c/00000000-0000-0000-0000-00005cfb00f8"
-          (reference "U18") (unit 1)
+          (reference "U11") (unit 1)
         )
       )
