File: KiCad OPEN ECU/rev. 02-2024/OEM_ECU.kicad_sch (KiCad schematic)
At the start: 47 parts, among them J1 TYPE-C-31-M-12, J6 RFShield_OnePiece, U1 ATSHA204A-MAHDA-T, U1 ESP32C3

Commit message: update
Other:
- added sheet WideBand O2 sensor (wideband_sensor.kicad_sch)
Changed lines of the file:
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@@
+    )
+  )
+  (sheet (at 79.8576 198.5772) (size 12.7 16.8656) (fields_autoplaced)
+    (stroke (width 0.1524) (type solid))
+    (fill (color 0 0 0 0.0000))
+    (property "Sheetname" "WideBand O2 sensor" (at 79.8576 197.8656 0)
+      (effects (font (size 1.27 1.27)) (justify left bottom))
+    )
+    (property "Sheetfile" "wideband_sensor.kicad_sch" (at 79.8576 216.0274 0)
+      (effects (font (size 1.27 1.27)) (justify left top))
+    )
+    (instances
+      (project "OEM_ECU"
+        (path "/ebe274a6-1c43-4fa2-9d2a-7756c5a7217c" (page "10"))
+      )
     )
   )

Commit message: update
Other:
- added sheet Serial UART (serial_uart.kicad_sch)
Changed lines of the file:
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@@
+    )
+  )
+  (sheet (at 83.9724 224.7646) (size 12.7 17.7546) (fields_autoplaced)
+    (stroke (width 0.1524) (type solid))
+    (fill (color 0 0 0 0.0000))
+    (property "Sheetname" "Serial UART" (at 83.9724 224.053 0)
+      (effects (font (size 1.27 1.27)) (justify left bottom))
+    )
+    (property "Sheetfile" "serial_uart.kicad_sch" (at 83.9724 243.1038 0)
+      (effects (font (size 1.27 1.27)) (justify left top))
+    )
+    (instances
+      (project "OEM_ECU"
+        (path "/ebe274a6-1c43-4fa2-9d2a-7756c5a7217c" (page "11"))
+      )
     )
   )
