File: KiCad OPEN ECU/rev. 02-2024/OEM_ECU.kicad_pcb (KiCad board)
At the start: 2 copper layers, 168.9 x 124.3 mm, 231 parts, among them IC1 MAX9926UAEE_V+, IC2 ZXMS6006DT8, IC3 ZXMS6006DT8, IC4 ZXMS6006DT8, J5 TYPE-C-31-M-12, Q2 Q_DUAL_NMOS_S1G1D2S2G2D1, Q3 Q_DUAL_NMOS_S1G1D2S2G2D1, SW1 219-2MSTR, SW2 219-2MSTR, SW3 219-2MSTR, SW4 219-2MSTR, U1 ESP32C3, U10 SP720, U11 KP234, U13 LMV324LIDT, U14 MPXH6400A, U16 ATSHA204A-MAHDA-T, U17 TC4424A, U18 MC33810, U19 MCP2562-E-SN, U2 MP1584EN, U20 LMV324LIDT, U21 AHT20, U22 TC4424A, U3 TC4424A, U4 TC4424A, U5 MC33810, U6 MC33810, U7 TC4424A, U8 TC4424A, U9 BMP280

Commit message: update
Parts:
- added CJC1: 2.2nF, Capacitor_SMD:C_0603_1608Metric, F.Cu at (121.6, 63.6)
- added CJC2: 100nF, Capacitor_SMD:C_0603_1608Metric, F.Cu at (108.8, 63.2)
- added CJC3: 100nF, Capacitor_SMD:C_0603_1608Metric, F.Cu at (112.4, 81.5)
- added CJC4: 100nF, Capacitor_SMD:C_0603_1608Metric, F.Cu at (112.4, 79.9)
- added CJC5: 100nF, Capacitor_SMD:C_0603_1608Metric, F.Cu at (123.2, 63.7)
- added CJC6: 100nF, Capacitor_SMD:C_0603_1608Metric, F.Cu at (119.8, 81.5)
- added CJC7: 33nF, Capacitor_SMD:C_0603_1608Metric, F.Cu at (119.8, 83.1)
- added CJC8: 33nF, Capacitor_SMD:C_0603_1608Metric, F.Cu at (107.2, 63.2)
- added CJQ1: AO3400A, Package_TO_SOT_SMD:SOT-23, F.Cu at (113.3, 61.5)
- added CJR1: 61R9, Resistor_SMD:R_0603_1608Metric, F.Cu at (119.2, 64.4)
- added CJR10: 100K, Resistor_SMD:R_0603_1608Metric, F.Cu at (118.3, 59.3)
- added CJR11: 4K7, Resistor_SMD:R_0603_1608Metric, F.Cu at (116.7, 59.4)
- added CJR2: 10K, Resistor_SMD:R_0603_1608Metric, F.Cu at (116.7, 63.6)
- added CJR3: 300R, Resistor_SMD:R_0603_1608Metric, F.Cu at (105.1, 72.3)
- added CJR4: 31K6, Resistor_SMD:R_0603_1608Metric, F.Cu at (110.4, 63.2)
- added CJR5: 4K7, Resistor_SMD:R_0603_1608Metric, F.Cu at (115.5, 79.9)
- added CJR6: 100K, Resistor_SMD:R_0603_1608Metric, F.Cu at (115.6, 81.9)
- added CJR7: 470K, Resistor_SMD:R_0603_1608Metric, F.Cu at (119.2, 61.8)
- added CJR8: 100K, Resistor_SMD:R_0603_1608Metric, F.Cu at (119.8, 79.9)
- added CJR9: 6K8, Resistor_SMD:R_0603_1608Metric, F.Cu at (113.8, 64.3)
- added U12: CJ125, AeonLabs_Automotive:CJ125 Wideband sensor, F.Cu at (114.6, 72.2)
- moved BT1 248.2 mm to (385.5, 78.2)
- moved C18 248.2 mm to (415.9, 97.0)
- moved C21 248.2 mm to (419.9, 97.1)
- moved C28 248.2 mm to (383.3, 108.9)
- moved JP1 248.2 mm to (404.2, 121.9)
- moved JP3 248.2 mm to (385.7, 94.3)
- moved MCU1 248.2 mm to (367.2, 72.4)
- moved MKC5 248.2 mm to (384.3, 70.0)
- moved MKC6 248.2 mm to (379.3, 70.0)
- moved MKCY2 248.2 mm to (376.7, 71.7)
- moved MKL2 248.2 mm to (381.0, 69.8)
- moved Q3 248.2 mm to (405.8, 84.7)
- moved R18 248.2 mm to (409.3, 97.0)
- moved R21 248.2 mm to (417.8, 97.0)
- moved R22 248.2 mm to (410.8, 97.0)
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Connections:
- U15 pad 25: unconnected-(U15-Pad25) -> LSU_VM
- U15 pad 26: unconnected-(U15-Pad26) -> LSU_HEAT-
- U15 pad 6: unconnected-(U15-Pad6) -> LSU_UN
- U15 pad 7: unconnected-(U15-Pad7) -> LSU_IA
- U15 pad 8: unconnected-(U15-Pad8) -> LSU_IP
Routing:
- net +12V: track 336.1 -> 499.5 mm, vias 11 -> 14
- net GND: track 1791.1 -> 1930.5 mm, vias 281 -> 284
- net +5V: track 205.1 -> 323.8 mm, vias 7 -> 10
- net UR: track 0.00 -> 50.7 mm, vias 0 -> 2
- net LSU_UN: track 0.00 -> 49.9 mm, vias 0 -> 3
- net LSU_VM: track 0.00 -> 43.9 mm
- net CJ_RST: track 0.00 -> 42.3 mm
- net Net-(U12-UP): track 0.00 -> 36.4 mm, vias 0 -> 2
- net LSU_IP: track 0.00 -> 27.5 mm, vias 0 -> 1
- net LSU_IA: track 0.00 -> 27.5 mm, vias 0 -> 1
- net LSU_HEAT-: track 0.00 -> 25.5 mm
- net UA: track 0.00 -> 25.3 mm
- net MOSI: track 124.1 -> 141.6 mm, vias 6 -> 7
- net CJ125_CS: track 0.00 -> 15.5 mm
- net MISO: track 124.0 -> 138.2 mm, vias 7 -> 8
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Other:
- board text added: "Injection and Ignition"
- board text added: "LSU 4.2/.9 O2 Sensor"
- board text added: "Power Supply"

Commit message: update
Parts:
- added CHC1: 1uF, Capacitor_SMD:C_0603_1608Metric, F.Cu at (117.2, 96.2)
- added CHC2: 1uF, Capacitor_SMD:C_0603_1608Metric, F.Cu at (117.9, 90.3)
- added CHC3: 1uF, Capacitor_SMD:C_0603_1608Metric, F.Cu at (117.2, 92.6)
- added J3: USB4120-03-C_REVA, AeonLabs_Connectors:USB-C Vertical GCT_USB4120-03-C_REVA, F.Cu at (111.3, 93.6)
- added PWR_FUSE1: Polyfuse, Fuse:Fuse_1206_3216Metric_Pad1.42x1.75mm_HandSolder, F.Cu at (120.6, 99.0)
- added U23: ~, AeonLabs_IC:CH9102F, F.Cu at (120.9, 93.8)
- added USB_PLUG_R3: 5k1, Resistor_SMD:R_0603_1608Metric, F.Cu at (108.1, 89.5)
- added USB_PLUG_R4: 5k1, Resistor_SMD:R_0603_1608Metric, F.Cu at (112.3, 97.6)
- added USB_PLYG_R2: 150K, Resistor_SMD:R_0603_1608Metric, F.Cu at (109.2, 97.5)
- moved CJC5 0.05 mm to (123.2, 63.6)
Routing:
- net +5V: track 323.8 -> 384.4 mm, vias 10 -> 11
- net GND: track 1930.5 -> 1973.6 mm, vias 284 -> 288
- net USB_5V0F: track 0.00 -> 29.9 mm
- net USB_D+: track 0.00 -> 16.8 mm
- net CJ_RST: track 42.3 -> 57.7 mm
- net USB_D-: track 0.11 -> 15.5 mm
- net UR: track 50.7 -> 66.0 mm
- net SCLK: track 132.3 -> 147.3 mm
- net MISO: track 138.2 -> 152.9 mm
- net MC33810_2-CS: track 50.1 -> 64.3 mm, vias 2 -> 3
- net CJ125_CS: track 15.5 -> 29.6 mm
- net MC33810_1-CS: track 66.4 -> 80.3 mm, vias 2 -> 3
- net MOSI: track 141.6 -> 155.4 mm
- net MC33810_3-CS: track 32.6 -> 46.4 mm, vias 2 -> 3
- net UA: track 25.3 -> 38.9 mm
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Other:
- board text added: "Firmware Update"
- board text added: "USB-C"
- board text removed: "USB-C EMS"

Commit message: update
Parts:
- removed C31: 0.1uF, Capacitor_SMD:C_0805_2012Metric
- removed JP1: Jumper_NO_Small, Jumper:SolderJumper-2_P1.3mm_Open_Pad1.0x1.5mm
- removed R50: 0R, Resistor_SMD:R_0805_2012Metric
- removed R54: 120R, Resistor_SMD:R_0805_2012Metric
- removed U19: MCP2562-E-SN, Package_SO:SOIC-8_3.9x4.9mm_P1.27mm
- added C7: 0.1uF, Capacitor_SMD:C_0805_2012Metric, F.Cu at (132.3, 100.0)
- added C8: 0.1uF, Capacitor_SMD:C_0805_2012Metric, F.Cu at (135.7, 96.0)
- added JP4: Jumper_NO_Small, Jumper:SolderJumper-2_P1.3mm_Open_Pad1.0x1.5mm, F.Cu at (131.3, 89.6)
- added R2: 120R, Resistor_SMD:R_0805_2012Metric, F.Cu at (133.8, 89.6)
- added U24: MCP2562-E_MF, AeonLabs_Automotive:MCP2562 DFN, F.Cu at (132.3, 96.0)
Connections:
- U15 pad 28: unconnected-(U15-Pad28) -> CAN_L
- U15 pad 9: unconnected-(U15-Pad9) -> CAN_H
Routing:
- net GND: track 1973.6 -> 2063.2 mm, vias 288 -> 290
- net CAN_H: track 22.4 -> 61.2 mm, vias 1 -> 2
- net CAN_L: track 24.5 -> 62.2 mm, vias 1 -> 0
- net ADC-Clamp-11: track 99.8 -> 73.8 mm
- net +3V3: track 627.5 -> 610.4 mm
- net ADC-Clamp-5: track 63.2 -> 49.3 mm
- net CAN_RXD: track 10.0 -> 16.4 mm
- net +5V: track 384.4 -> 390.4 mm, vias 11 -> 13
- net CAN_TXD: track 11.1 -> 14.8 mm
- net Net-(U19-STBY): track 2.90 -> 0.00 mm
- net Net-(JP4-Pad2): track 0.00 -> 2.14 mm
- net Net-(JP1-Pad2): track 2.01 -> 0.00 mm
Other:
- board text added: "120R"
- board text added: "TWAI"

Commit message: update
Parts:
- removed J5: TYPE-C-31-M-12, Connector_USB:USB_C_Receptacle_HRO_TYPE-C-31-M-12
- removed MKR2, MKR3: 33R, Resistor_SMD:R_0603_1608Metric
- removed UART_CON2: UART_CONN, AeonLabs_Connectors:SOIC_clipProgSmall
- removed USB_PLUG_R1, USB_PLUG_R2: 5k1, Resistor_SMD:R_0603_1608Metric
- removed USB_PLYG_R1: 150K, Resistor_SMD:R_0603_1608Metric
- moved AUC1 261.9 mm to (383.0, 166.9)
- moved EC14 261.9 mm to (391.2, 164.7)
- moved EC15 261.9 mm to (390.5, 171.7)
- moved EC17 261.9 mm to (400.9, 163.8)
- moved EC2 261.9 mm to (391.9, 160.1)
- moved EC3 261.9 mm to (403.5, 164.5)
- moved EC5 261.9 mm to (403.1, 170.4)
- moved EC6 261.9 mm to (388.4, 160.3)
- moved EC7 261.9 mm to (388.4, 164.1)
- moved EC8 261.9 mm to (398.2, 161.4)
- moved EC9 261.9 mm to (397.1, 158.4)
- moved ECY1 261.9 mm to (394.5, 160.0)
- moved ECY2 261.9 mm to (403.3, 167.4)
- moved ER2 261.9 mm to (400.7, 169.0)
- moved ER3 261.9 mm to (388.9, 170.1)
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Connections:
- G*** pad 1: (no net) -> GNDA
Routing:
- net GNDA: track 53.3 -> 131.1 mm, vias 256 -> 301
- net GND: vias 290 -> 288
Other:
- board text added: "Edge length = 124.3mm (Incl curves)"
- board text added: "Edge length = 169mm (Incl curves)"
- board text removed: "CAN"
- board text removed: "Edge length = 117.2mm (Incl curves)"
- board text removed: "Edge length = 148.9mm (Incl curves)"
- board text removed: "UART EMS"
