File: KiCad OPEN ECU/rev. 02-2024/inputs.kicad_sch (KiCad schematic)
At the start: 41 parts, among them SW3 219-2MSTR, U10 SP720, U11 KP234, U13 LMV324LIDT, U14 MPXH6400A

Commit message: update
Changed lines of the file:
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@@
   )
   (symbol (lib_id "AeonLabs_Automotive:KP234") (at 133.35 46.99 0) (unit 1)
-    (in_bom yes) (on_board yes) (dnp no) (fields_autoplaced)
+    (in_bom yes) (on_board yes) (dnp no)
     (property "Reference" "U11" (at 121.3612 44.45 0)
       (effects (font (size 1.27 1.27)) (justify right))
@@
       (effects (font (size 1.27 1.27)) (justify right))
     )
-    (property "Footprint" "AeonLabs_Automotive:kp234 barometric sensor" (at 121.3612 49.53 0)
+    (property "Footprint" "AeonLabs_Automotive:kp234 barometric sensor" (at 157.988 57.5056 0)
       (effects (font (size 1.27 1.27)) (justify right))
     )
