File: KiCad Dual Band Antenna/rev. 03-2024/dual_band_antenna.kicad_sch (KiCad schematic)
At the start: 0 parts

Commit message: Add files via upload
Other:
- note added: "There's no circuit schematics"
Changed lines of the file:
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@@
-(kicad_sch (version 20240101) (generator "eeschema") (generator_version "8.99")
-  (paper "A4")
-  (symbol_instances)
+(kicad_sch
+	(version 20240101)
+	(generator "eeschema")
+	(generator_version "8.99")
+	(paper "A4")
+	(text "There's no circuit schematics"
+		(exclude_from_sim no)
+		(at 144.272 96.266 0)
+		(effects
+			(font
+				(size 5.08 5.08)
+			)
+		)
+	)
+	(sheet_instances
+		(path "/"
+			(page "1")
+		)
+	)
 )
