File: KiCad Dual Band Antenna/rev. 03-2024/dual_band_antenna.kicad_pcb (KiCad board)
At the start: 2 copper layers, 114.4 x 47.1 mm, 5 parts

Commit message: Add files via upload
Parts:
- moved G*** 0.26 mm to (149.7, 97.2)
Other:
- outline, holes or cut-outs redrawn
